File: The_Grid_PCB/The_Grid_PCB.kicad_pcb (KiCad board)
At the start: 2 copper layers, 115 x 60 mm, 111 parts, among them J1 TC2050, J10 Screw_Terminal_01x02, J11 Screw_Terminal_01x02, J12 Screw_Terminal_01x02, J13 Screw_Terminal_01x02, J14 Screw_Terminal_01x02, J15 Screw_Terminal_01x02, J16 Screw_Terminal_01x02, J17 Screw_Terminal_01x02, J2 Screw_Terminal_01x02, J3 Screw_Terminal_01x03, J4 Screw_Terminal_01x03, J5 Screw_Terminal_01x02, J6 Screw_Terminal_01x02, J7 Screw_Terminal_01x02, J8 Screw_Terminal_01x02, J9 Screw_Terminal_01x02, Q1 AO3400A, Q10 AO3400A, Q11 AO3400A, Q12 AO3400A, Q2 AO3400A, Q3 AO3400A, Q4 AO3400A, Q5 AO3400A, Q6 AO3400A, Q7 AO3400A, Q8 AO3400A, Q9 AO3400A, U1 STM32F030C8Tx, U2 SN65HVD485EDR, U3 TPS54331DR, U4 AMS1117-3.3, X1 X322516MLB4SI

Commit message: rev1 pcb sent to prod
Parts:
- removed the C1 at (129.8, 105.6)
- removed C19: 10uF, PCM_JLCPCB:C_0603
- removed the C2 at (130.0, 103.5)
- removed C22: 22uF, PCM_JLCPCB:C_0603
- removed C24: 100nF, PCM_JLCPCB:C_0805
- removed the C3 at (125.5, 104.9)
- removed the C4 at (125.5, 110.9)
- removed the C5 at (132.2, 102.8)
- removed the C6 at (139.4, 114.2)
- removed the C7 at (130.2, 110.8)
- removed the C8 at (129.0, 113.2)
- removed the J1 at (113.6, 107.5)
- removed the R3 at (128.4, 109.8)
- removed the R4 at (135.5, 100.0)
- removed U4: AMS1117-3.3, Package_TO_SOT_SMD:SOT-223-3_TabPin2
- removed X1: X322516MLB4SI, PCM_JLCPCB:OSC-SMD_4P-L3.2-W2.5-BL
- added TP5: 5V, TestPoint:TestPoint_THTPad_D2.0mm_Drill1.0mm, F.Cu at (160.3, 111.0)
- U1: value STM32F030C8Tx -> STM32 Blue Pill; footprint Package_QFP:LQFP-48_7x7mm_P0.5mm -> BluePill_Header:STM32BluePill
- moved TP4 17.9 mm to (173.6, 111.0)
- moved TP3 17.9 mm to (166.9, 110.9)
- moved R7 11.2 mm to (168.7, 92.2), turned to 0 degrees
- moved C12 7.40 mm to (133.2, 92.8)
- moved C11 7.40 mm to (130.3, 92.8)
- moved C1 7.40 mm to (145.2, 81.5)
- moved C10 7.40 mm to (130.2, 78.0)
- moved C3 7.40 mm to (150.2, 81.5)
- moved C4 7.40 mm to (156.2, 80.0)
- moved C5 7.40 mm to (147.8, 81.5)
- moved C6 7.40 mm to (142.8, 81.5)
- moved C7 7.40 mm to (142.8, 77.5)
- moved C8 7.40 mm to (133.2, 84.0)
- moved C9 7.40 mm to (124.8, 78.0)
- moved D4 7.40 mm to (135.8, 87.0)
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- renumbered C9 to C1, C18 to C10, C20 to C11, C21 to C12, C23 to C13, C25 to C14, C10 to C2, C11 to C3, C12 to C4, C13 to C5, C14 to C6, C15 to C7, C16 to C8, C17 to C9, J2 to J1, J11 to J10, J12 to J11, J13 to J12, J14 to J13, J15 to J14, J16 to J15, J17 to J16, J3 to J2, J4 to J3, J5 to J4, J6 to J5, J7 to J6, J8 to J7, J9 to J8, J10 to J9, R12 to R10, R13 to R11, R14 to R12, R15 to R13, R16 to R14, R17 to R15, R18 to R16, R19 to R17, R20 to R18, R21 to R19, R22 to R20, R23 to R21, R24 to R22, R25 to R23, R26 to R24, R27 to R25, R28 to R26, R29 to R27, R30 to R28, R31 to R29, R5 to R3, R32 to R30, R33 to R31, R34 to R32, R35 to R33, R36 to R34, R37 to R35, R38 to R36, R39 to R37, R40 to R38, R41 to R39, R6 to R4, R42 to R40, R43 to R41, R7 to R5, R8 to R6, R9 to R7, R10 to R8, R11 to R9
Connections:
- U1 pad 11: unconnected-(U1-PA1-Pad11) -> /R2
- U1 pad 12: /VCP_RX_MCU_TX -> /B1
- U1 pad 13: /B1 -> /G1
- U1 pad 14: /R2 -> /R1
- U1 pad 15: unconnected-(U1-PA5-Pad15) -> /TX
- U1 pad 16: /G2 -> /RX
- U1 pad 17: /B2 -> unconnected-(U1-RST-Pad17)
- U1 pad 18: /R4 -> +3.3V
- U1 pad 19: /G4 -> GND
- U1 pad 20: /Microswitch1 -> GND
- U1 pad 21: /DE -> unconnected-(U1-PB12-Pad21)
- U1 pad 23: GND -> unconnected-(U1-PB14-Pad23)
- U1 pad 24: +3.3V -> unconnected-(U1-PB15-Pad24)
- U1 pad 27: /B4 -> unconnected-(U1-PA10-Pad27)
- U1 pad 29: /R3 -> unconnected-(U1-PA12-Pad29)
- U1 pad 30: unconnected-(U1-PA9-Pad30) -> /Microswitch1
- U1 pad 31: /G3 -> /Microswitch2
- U1 pad 32: /B3 -> /Microswitch3
- U1 pad 33: unconnected-(U1-PA12-Pad33) -> /Microswitch4
- U1 pad 34: /SWDIO -> /G2
- U1 pad 35: unconnected-(U1-PF6-Pad35) -> /B2
- U1 pad 36: unconnected-(U1-PF7-Pad36) -> /R4
- U1 pad 37: /SWCLK -> /G4
- U1 pad 38: /VCP_TX_MCU_RX -> +5V
- U1 pad 39: /Microswitch4 -> GND
- U1 pad 40: /Microswitch3 -> +3.3V
- U1 pad 5: /OSC_IN -> /B3
- U1 pad 6: /OSC_OUT -> /G3
- U1 pad 7: /nRST -> /R3
- U1 pad 8: GND -> /B4
- U1 pad 9: +3.3V -> /DE
Routing:
- net +24V: track 257.8 -> 52.3 mm
- net GND: track 162.3 -> 23.5 mm, vias 75 -> 506
- net /VCP_RX_MCU_TX: track 34.4 -> 0.00 mm
- net /VCP_TX_MCU_RX: track 33.3 -> 0.00 mm, vias 2 -> 0
- net /nRST: track 29.9 -> 0.00 mm, vias 2 -> 0
- net /SWCLK: track 29.0 -> 0.00 mm, vias 2 -> 0
- net /SWDIO: track 27.8 -> 0.00 mm, vias 2 -> 0
- net +3.3V: track 193.1 -> 165.3 mm, vias 7 -> 2
- net /RX: track 42.9 -> 66.7 mm
- net /TX: track 37.5 -> 60.5 mm
- net +5V: track 86.0 -> 104.0 mm
- net /Microswitch2: track 27.9 -> 14.1 mm, vias 1 -> 0
- net /R1: track 37.2 -> 24.9 mm
- net /G4: track 46.5 -> 35.1 mm
- net /G1: track 36.1 -> 24.9 mm
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- added copper zone on B.Cu, net +5V
- removed copper zone on B.Cu, net +3.3V
- removed copper zone on F.Cu, net +3.3V
- removed copper zone on F.Cu, net /RSA
- removed copper zone on F.Cu, net /RSB
Other:
- board text added: "+24V"
- board text added: "24V"
- board text added: "5V"
- board text added: "B1"
- board text added: "B2"
- board text added: "B3"
- board text added: "B4"
- board text added: "G1"
- board text added: "G2"
- board text added: "G3"
- board text added: "G4"
- board text added: "R1"
- board text added: "R2"
- board text added: "R3"
- board text added: "R4"
- board text added: "RSA"
- board text added: "RSB"
