File: The_Grid_PCB/pixel_mosfets.kicad_sch (KiCad schematic)
At the start: 11 parts, among them J1 Screw_Terminal_01x02, J2 Screw_Terminal_01x02, Q1 AO3400A, Q2 AO3400A, Q3 AO3400A

Commit message: pcb iter 1 done
Parts:
- J10: renamed from J1; footprint TerminalBlock_4Ucon:TerminalBlock_4Ucon_1x02_P3.50mm_Vertical -> TerminalBlock_4Ucon:TerminalBlock_4Ucon_1x02_P3.50mm_Horizontal; LCSC (none) -> C695629
- J11: renamed from J2; footprint TerminalBlock_4Ucon:TerminalBlock_4Ucon_1x02_P3.50mm_Vertical -> TerminalBlock_4Ucon:TerminalBlock_4Ucon_1x02_P3.50mm_Horizontal; LCSC (none) -> C695629
- renumbered R8 to R18, R9 to R19, R11 to R20, R10 to R21, R13 to R22, R12 to R23
Connections:
- net B: no longer R23.1
- net G: no longer R21.1
- net R: no longer R19.1
- net at Q1.1 (G), R18.2: now also R19.1
- net at Q3.1 (G), R22.2: now also R23.1
- net at Q2.1 (G), R20.2: now also R21.1
Other:
- moved on the sheet: R18, R19, R20, R21, R22, R23

Commit message: update wiring diagram again sob
Parts:
- renumbered R18 to R20, R19 to R21, R20 to R22, R21 to R23, R22 to R24, R23 to R25

Commit message: rev1 pcb sent to prod
Parts:
- renumbered J11 to J10, J10 to J9, R20 to R18, R21 to R19, R22 to R20, R23 to R21, R24 to R22, R25 to R23
