File: The_Grid_PCB/pixel_mosfets.kicad_sch (KiCad schematic)
At the start: 11 parts, among them J10 Screw_Terminal_01x02, J9 Screw_Terminal_01x02, Q1 AO3400A, Q2 AO3400A, Q3 AO3400A

Commit message: rev2 minus silkscreen
Parts:
- renumbered R18 to R17, R19 to R18, R20 to R19, R21 to R20, R22 to R21, R23 to R22
