File: The_Grid_PCB/The_Grid_PCB.kicad_sch (KiCad schematic)
At the start: 52 parts, among them J1 Screw_Terminal_01x02, J2 Screw_Terminal_01x03, J3 Screw_Terminal_01x03, J4 Screw_Terminal_01x02, J5 Screw_Terminal_01x02, J6 Screw_Terminal_01x02, J7 Screw_Terminal_01x02, J8 Screw_Terminal_01x02, U1 STM32 Blue Pill, U2 SN65HVD485EDR, U3 TPS54331DR

Commit message: pcb impedence matching, switch cap filtering, mounting holes, silkscreen updates
Parts:
- added C10, C11, C16, C17, C3: 100nF, PCM_JLCPCB:C_0603, symbol PCM_JLCPCB-Capacitors:0603,100nF
- renumbered C9 to C12, C10 to C13, C11 to C14, C12 to C15, C13 to C18, C14 to C19, C3 to C4, C4 to C5, C5 to C6, C6 to C7, C7 to C8, C8 to C9
Connections:
- net +5V: now also C3.1
- net GND: now also C10.2, C11.2, C16.2, C17.2, C3.2
- net Microswitch1: now also C10.1
- net Microswitch2: now also C11.1
- net Microswitch3: now also C16.1
- net Microswitch4: now also C17.1
- net RSA renamed RS+
- net RSB renamed RS-
Other:
- moved on the sheet: C2

Commit message: rev2 minus silkscreen
Parts:
- removed D2: LED, PCM_JLCPCB:D_0603, symbol Device:LED
- removed R1: 220Ω, PCM_JLCPCB:R_0603, symbol PCM_JLCPCB-Resistors:0603,220Ω
- removed R2: 1.5kΩ, PCM_JLCPCB:R_0603, symbol PCM_JLCPCB-Resistors:0603,1.5kΩ
- added R1: 560Ω, PCM_JLCPCB:R_0603, symbol PCM_JLCPCB-Resistors:0603,560Ω
- renumbered D3 to D2, D4 to D3, R11 to R10, R12 to R11, R13 to R12, R14 to R13, R15 to R14, R16 to R15, R17 to R16, R3 to R2, R4 to R3, R5 to R4, R6 to R5, R7 to R6, R8 to R7, R9 to R8, R10 to R9
Connections:
- net GND: now also R1.2
- net at D1.1 (K): now also R1.1
Other:
- note removed: "24V Power indication LED"
- moved on the sheet: D1
