File: The_Grid_PCB/The_Grid_PCB.kicad_sch (KiCad schematic)
At the start: 55 parts, among them J1 Screw_Terminal_01x02, J2 Screw_Terminal_01x03, J3 Screw_Terminal_01x03, J4 Screw_Terminal_01x02, J5 Screw_Terminal_01x02, J6 Screw_Terminal_01x02, J7 Screw_Terminal_01x02, J8 Screw_Terminal_01x02, U1 STM32 Blue Pill, U2 SN65HVD485EDR, U3 TPS54331DR

Commit message: pcb rev2 sent to fab
Parts:
- U2: value SN65HVD485EDR -> THDV1520; Arrow Part Number SN65HVD485EDR -> (none); Arrow Price/Stock https://www.arrow.com/en/products/sn65hvd485edr/texas-instr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 -> (none); LCSC C27899 -> C882408; Manufacturer_Part_Number SN65HVD485EDR -> THDV1520; Mouser Part Number 595-SN65HVD485EDR -> (none); Mouser Price/Stock https://www.mouser.co.uk/ProductDetail/Texas-Instruments/SN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 -> (none)
Connections:
- net GND: no longer U1.20 (GND)
- no-connect marks 15 -> 16
Other:
- note added: "In the alibaba version of these chips Pin20 is actually 5v!!!"
Changed lines of the file:
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@@
 		)
 	)
+	(text "In the alibaba version of these \nchips Pin20 is actually 5v!!!"
+		(exclude_from_sim no)
+		(at 134.112 48.768 0)
+		(effects
+			(font
+				(size 1.27 1.27)
+			)
+		)
+	)
 	(text "For start node - connect to devboard \nto use RS-485 Transceiver\n"
 		(exclude_from_sim no)
@@
 	)
 	(junction
-		(at 107.95 50.8)
-		(diameter 0)
-		(color 0 0 0 0)
-	)
-	(junction
 		(at 306.07 48.26)
 		(diameter 0)
@@
 	)
 	(no_connect
+		(at 107.95 50.8)
+	)
+	(no_connect
 		(at 226.06 55.88)
 	)
@@
 	(wire
 		(pts
-			(xy 107.95 50.8) (xy 107.95 53.34)
-		)
-		(stroke
-			(width 0)
-			(type default)
-		)
-	)
-	(wire
-		(pts
 			(xy 256.54 53.34) (xy 261.62 53.34)
 		)
@@
 	(wire
 		(pts
-			(xy 107.95 50.8) (xy 116.84 50.8)
+			(xy 107.95 53.34) (xy 116.84 53.34)
 		)
 		(stroke
@@
 	(wire
 		(pts
-			(xy 116.84 50.8) (xy 116.84 58.42)
+			(xy 116.84 53.34) (xy 116.84 58.42)
 		)
 		(stroke
@@
 			)
 		)
-		(property "Value" "SN65HVD485EDR"
+		(property "Value" "THDV1520"
 			(at 201.93 111.76 0)
 			(show_name no)
@@
 			)
 		)
-		(property "Datasheet" "http://www.ti.com/lit/gpn/sn65hvd485e"
+		(property "Datasheet" "https://www.ti.com/lit/ds/symlink/thvd1520.pdf?ts=1784928696084&ref_url=https%253A%252F%252Fwww.ti.com"
 			(at 210.82 311.76 0)
 			(hide yes)
@@
 			)
 		)
-		(property "Manufacturer_Part_Number" "SN65HVD485EDR"
+		(property "Manufacturer_Part_Number" "THDV1520"
 			(at 210.82 711.76 0)
 			(hide yes)
@@
 			)
 		)
-		(property "Mouser Part Number" "595-SN65HVD485EDR"
-			(at 210.82 811.76 0)
-			(hide yes)
-			(show_name no)
-			(do_not_autoplace no)
-			(effects
-				(font
-					(size 1.27 1.27)
-				)
-				(justify left top)
-			)
-		)
-		(property "Mouser Price/Stock" "https://www.mouser.co.uk/ProductDetail/Texas-Instruments/SN65HVD485EDR?qs=QViXGNcIEAu4qPXpVA5%252B5Q%3D%3D"
-			(at 210.82 911.76 0)
-			(hide yes)
-			(show_name no)
-			(do_not_autoplace no)
-			(effects
-				(font
-					(size 1.27 1.27)
-				)
-				(justify left top)
-			)
-		)
-		(property "Arrow Part Number" "SN65HVD485EDR"
-			(at 210.82 1011.76 0)
-			(hide yes)
-			(show_name no)
-			(do_not_autoplace no)
-			(effects
-				(font
-					(size 1.27 1.27)
-				)
-				(justify left top)
-			)
-		)
-		(property "Arrow Price/Stock" "https://www.arrow.com/en/products/sn65hvd485edr/texas-instruments?region=nac"
-			(at 210.82 1111.76 0)
-			(hide yes)
-			(show_name no)
-			(do_not_autoplace no)
-			(effects
-				(font
-					(size 1.27 1.27)
-				)
-				(justify left top)
-			)
-		)
-		(property "LCSC" "C27899"
+		(property "LCSC" "C882408"
 			(at 189.23 116.84 0)
 			(hide yes)
